Commit message: mods

File: urdf/model.urdf (robot description, URDF)
Before this commit: robot RCV, 2 links, 1 joints
Links:
- link base: geometry collision box size=4 2 .5; visual box size=4 2 .5
- link camera1: geometry collision box size=.065 .25 .065; visual box size=.065 .25 .065

Commit message: model dimensions changed

File: urdf/model.urdf (robot description, URDF)
Before this commit: robot RCV, 2 links, 1 joints
Links:
- removed link base
- added link base_link; collision box size=2.4 1.6 .5; visual box size=2.4 1.6 .5
Joints:
- joint camera1connect: parent base -> base_link

Commit message: now camera is in front

File: urdf/model.urdf (robot description, URDF)
Before this commit: robot RCV, 2 links, 1 joints
Joints:
- joint camera1connect: origin xyz=0 0 1.5 rpy=0 0 0 -> xyz=1.4 0 0 rpy=0 0 0
